File: sEMG_v1.kicad_pcb (KiCad board)
At the start: 2 copper layers, 42.1 x 31.9 mm, 39 parts, among them J1 AudioJack3_SwitchTR, J2 Jumper_3_Bridged12, J3 Conn_01x10

Commit message: update v1
Parts:
- added ?: , , F.Cu at (100.0, 111.2)
- added ?: , , F.Cu at (139.8, 140.7)
- added ?: , , F.Cu at (100.1, 140.8)
- added ?: , , F.Cu at (139.8, 111.2)
- added R16: 22k, course_kicad_ecp_footprint:RC0603JR-070RL, F.Cu at (107.8, 137.2)
- added R17: 22k, course_kicad_ecp_footprint:RC0603JR-070RL, F.Cu at (109.3, 137.2)
- moved R15 15.5 mm to (109.5, 120.6)
- moved D1 8.04 mm to (115.7, 116.4), turned to 90 degrees
- moved R1 3.30 mm to (114.0, 116.6), turned to 90 degrees
- moved J2 3.14 mm to (120.0, 118.4), turned to 90 degrees
- moved R2 1.56 mm to (111.9, 118.9)
- moved C16 1.39 mm to (110.8, 137.1)
- moved C15 1.33 mm to (114.4, 137.1)
- moved R14 1.33 mm to (112.6, 137.1)
- moved R10 1.32 mm to (120.4, 137.1)
- moved R11 1.32 mm to (119.0, 137.1)
- moved R12 1.32 mm to (115.9, 137.1)
- moved R13 1.32 mm to (122.0, 137.1)
- moved R9 1.32 mm to (117.5, 137.1)
- moved C10 0.46 mm to (118.5, 123.5)
- moved C11 0.46 mm to (116.7, 123.7)
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Connections:
- J3 pad 10: GND -> /~{DRDY}
- J3 pad 2: /~{PWDN/RESET} -> GND
- J3 pad 3: /START -> /~{PWDN/RESET}
- J3 pad 4: /~{DRDY} -> /START
- J3 pad 5: /~{CS} -> /CLK
- J3 pad 6: /DIN -> /~{CS}
- J3 pad 7: /DOUT -> /DIN
- J3 pad 9: /CLK -> /DOUT
- U1 pad 25: unconnected-(U1-GPIO2/RCLK2-Pad25) -> Net-(U1-GPIO2/RCLK2)
- U1 pad 26: unconnected-(U1-GPIO1/RCLK1-Pad26) -> Net-(U1-GPIO1/RCLK1)
- U1 pad 31: unconnected-(U1-RESP_MODP/IN3P-Pad31) -> /AVDD
- U1 pad 32: unconnected-(U1-RESP_MODN/IN3N-Pad32) -> /AVDD
- U1 pad 5: unconnected-(U1-IN2N-Pad5) -> /AVDD
- U1 pad 6: unconnected-(U1-IN2P-Pad6) -> /AVDD
Routing:
- net GND: track 48.3 -> 18.2 mm, vias 5 -> 69
- net /AVSS: track 52.2 -> 33.0 mm, vias 7 -> 8
- net /AVDD: track 32.3 -> 43.0 mm, vias 3 -> 2
- net /~{PWDN/RESET}: track 19.7 -> 13.5 mm, vias 1 -> 0
- net Net-(U1-GPIO2/RCLK2): track 0.00 -> 5.30 mm
- net /TN: track 22.8 -> 18.1 mm
- net Net-(U1-GPIO1/RCLK1): track 0.00 -> 4.71 mm
- net /VCC3V3: track 40.2 -> 35.7 mm, vias 4 -> 2
- net /CLK: track 14.1 -> 9.59 mm, vias 1 -> 0
- net /~{DRDY}: track 15.5 -> 12.2 mm, vias 0 -> 1
- net /DOUT: track 8.83 -> 11.9 mm, vias 1 -> 0
- net Net-(U1-RLDINV): track 7.30 -> 5.01 mm
- net Net-(U1-RLDOUT): track 4.29 -> 5.87 mm
- net Net-(U1-RLDIN/RLDREF): track 3.44 -> 4.99 mm
- net Net-(U1-VCAP2): track 5.28 -> 3.90 mm
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