File: sEMG_v1.kicad_sch (KiCad schematic)
At the start: 39 parts, among them J1 AudioJack3_SwitchTR, J2 Jumper_3_Bridged12, J3 Conn_01x10

Commit message: update v1
Parts:
- added R16, R17: 22k, course_kicad_ecp_footprint:RC0603JR-070RL, symbol Device:R
Connections:
- net AVDD: now also U1.31 (RESP_MODP/IN3P), U1.32 (RESP_MODN/IN3N), U1.5 (IN2N), U1.6 (IN2P)
- net CLK: now also J3.5 (Pin_5); no longer J3.9 (Pin_9)
- net DIN: now also J3.7 (Pin_7); no longer J3.6 (Pin_6)
- net DOUT: now also J3.9 (Pin_9); no longer J3.7 (Pin_7)
- net GND: now also J3.2 (Pin_2), R16.2, R17.2; no longer J3.10 (Pin_10)
- net START: now also J3.4 (Pin_4); no longer J3.3 (Pin_3)
- net ~{CS}: now also J3.6 (Pin_6); no longer J3.5 (Pin_5)
- net ~{DRDY}: now also J3.10 (Pin_10); no longer J3.4 (Pin_4)
- net ~{PWDN/RESET}: now also J3.3 (Pin_3); no longer J3.2 (Pin_2)
- net at U1.25 (GPIO2/RCLK2): now also R16.1
- net at U1.26 (GPIO1/RCLK1): now also R17.1
- no-connect marks 6 -> 0
