File: sEMG_v1.kicad_sch (KiCad schematic)
At the start: 41 parts, among them J1 Conn_01x10

Commit message: Update sEMG_v1 project
Parts:
- R14, R5, R6, R7, R8: value 1M -> 10M
Changed lines of the file:
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@@
 			)
 		)
-		(property "Value" "1M"
+		(property "Value" "10M"
 			(at 203.2 92.71 90)
 			(show_name no)
@@
 			)
 		)
-		(property "Value" "1M"
+		(property "Value" "10M"
 			(at 86.36 90.1699 0)
 			(show_name no)
@@
 			)
 		)
-		(property "Value" "1M"
+		(property "Value" "10M"
 			(at 86.36 113.0299 0)
 			(show_name no)
@@
 			)
 		)
-		(property "Value" "1M"
+		(property "Value" "10M"
 			(at 86.36 124.4599 0)
 			(show_name no)
@@
 			)
 		)
-		(property "Value" "1M"
+		(property "Value" "10M"
 			(at 86.36 78.7399 0)
 			(show_name no)
