File: _restore_backup_2026-06-14T18-33-25-370/sEMG_v1.kicad_sch (KiCad schematic)
At the start: 41 parts, among them J1 Conn_01x10

Commit message: completed sEMG v1.0
Parts:
- D1: Link MY_FOOTPRINTS:pad-1x10 -> (none)
- J1: footprint MY_FOOTPRINTS:SJ2-3593D-SMT-TR -> MY_FOOTPRINTS:pad-1x10
- J3: footprint MY_FOOTPRINTS:pad-1x10 -> MY_FOOTPRINTS:SJ2-3593D-SMT-TR
- R10, R11, R12, R13, R15, R2, R3, R4, R9: footprint MY_FOOTPRINTS:R_0603 -> MY_FOOTPRINTS:R0603
Changed lines of the file:
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@@
 			)
 		)
-		(property "Footprint" "MY_FOOTPRINTS:R_0603"
+		(property "Footprint" "MY_FOOTPRINTS:R0603"
 			(at 212.598 68.58 90)
 			(hide yes)
@@
 			)
 		)
-		(property "Footprint" "MY_FOOTPRINTS:SJ2-3593D-SMT-TR"
+		(property "Footprint" "MY_FOOTPRINTS:pad-1x10"
 			(at 25.4 97.79 0)
 			(hide yes)
@@
 			)
 		)
-		(property "Footprint" "MY_FOOTPRINTS:R_0603"
+		(property "Footprint" "MY_FOOTPRINTS:R0603"
 			(at 45.72 119.888 90)
 			(hide yes)
@@
 			)
 		)
-		(property "Footprint" "MY_FOOTPRINTS:R_0603"
+		(property "Footprint" "MY_FOOTPRINTS:R0603"
 			(at 224.79 83.058 90)
 			(hide yes)
@@
 			)
 		)
-		(property "Footprint" "MY_FOOTPRINTS:R_0603"
+		(property "Footprint" "MY_FOOTPRINTS:R0603"
 			(at 93.98 27.432 90)
 			(hide yes)
@@
 			)
 		)
-		(property "Footprint" "MY_FOOTPRINTS:R_0603"
+		(property "Footprint" "MY_FOOTPRINTS:R0603"
 			(at 218.948 68.58 90)
 			(hide yes)
@@
 			)
 		)
-		(property "Footprint" "MY_FOOTPRINTS:pad-1x10"
+		(property "Footprint" "MY_FOOTPRINTS:SJ2-3593D-SMT-TR"
 			(at 217.17 137.16 0)
 			(hide yes)
@@
 			)
 		)
-		(property "Footprint" "MY_FOOTPRINTS:R_0603"
+		(property "Footprint" "MY_FOOTPRINTS:R0603"
 			(at 103.378 129.54 90)
 			(hide yes)
@@
 			)
 		)
-		(property "Footprint" "MY_FOOTPRINTS:R_0603"
+		(property "Footprint" "MY_FOOTPRINTS:R0603"
 			(at 204.47 77.978 90)
 			(hide yes)
@@
 			)
 		)
-		(property "Footprint" "MY_FOOTPRINTS:R_0603"
+		(property "Footprint" "MY_FOOTPRINTS:R0603"
 			(at 45.72 85.598 90)
 			(hide yes)
@@
 			)
 		)
-		(property "Link" "MY_FOOTPRINTS:pad-1x10"
-			(at 87.63 46.99 90)
-			(hide yes)
-			(show_name no)
-			(do_not_autoplace no)
-			(effects
-				(font
-					(size 1.27 1.27)
-				)
-			)
-		)
 		(pin "1"
 		)
@@
 			)
 		)
-		(property "Footprint" "MY_FOOTPRINTS:R_0603"
+		(property "Footprint" "MY_FOOTPRINTS:R0603"
 			(at 204.47 83.058 90)
 			(hide yes)
