File: _restore_backup_2026-06-15T01-37-18-669/sEMG_v1.kicad_pcb (KiCad board)
At the start: 2 copper layers, 42.2 x 33.9 mm, 46 parts, among them J1 Conn_01x10

Commit message: completed sEMG v1.0
Parts:
- removed G***: LOGO, MY_FOOTPRINTS:logo_trilucas3
- moved ? 1.16 mm to (139.7, 141.3)
- moved ? 1.09 mm to (100.3, 141.3)
Other:
- board size 42.2 x 33.9 mm -> 42.2 x 32.6 mm
- board text removed: "sEMG v1.0"
